Commit message: removes dual structure for korus v2 and v3 (v2 wont use this code base)

File: korus_meta/resources/urdf/components/diff_drive_base.urdf.xacro (robot description, xacro)
@@ -57,5 +57,5 @@
 		  <visual>
 		    <geometry>
-		      <cylinder length="0.299" radius="0.278"/>
+		      <mesh filename="package://korus_meta/resources/meshes/base_test_model.dae" />
 		    </geometry>
 		    <origin xyz="0.0 0.0 0.1045" rpy="0 0 0"/>

File: korus_meta/resources/urdf/korus_all.urdf.xacro (robot description, xacro)
@@ -1,12 +1,15 @@
 <?xml version="1.0" ?>
-<robot name="korus_v3" xmlns:xacro="http://www.ros.org/wiki/xacro">
-  <xacro:include filename="$(find korus_meta)/resources/urdf/components/diff_drive_base.urdf.xacro"/>
+<robot name="korus" xmlns:xacro="http://www.ros.org/wiki/xacro">
+  <xacro:include filename="$(find korus_meta)/resources/urdf/components/omni_drive_base.urdf.xacro"/>
   <xacro:include filename="$(find korus_meta)/resources/urdf/components/upper_body.urdf.xacro"/>
   <xacro:include filename="$(find korus_meta)/resources/urdf/components/arm.urdf.xacro"/>
+  <xacro:include filename="$(find korus_meta)/resources/urdf/environment/table.urdf.xacro"/>
   <!-- ************************ Base model ************************* -->
-  <xacro:diff_drive_base parent="base_footprint" body_mount_link="base_link"/>
+  <xacro:omni_drive_base parent="local_manip_start" body_mount_link="base_link"/>
   <!-- ************************ Body model ************************* -->
   <xacro:upper_body body_mount_link="base_link" arm_mount_link="torso_lift_link"/>
   <!-- ************************ Arm model ************************* -->
   <xacro:arm arm_mount_link="torso_lift_link"/>
+  <!-- ************************ Table model ************************* -->
+  <xacro:table parent="local_manip_start"/>
 </robot>

File: korus_meta/resources/urdf/korus_diff_drive.urdf.xacro (robot description, xacro)
@@ -1,15 +1,12 @@
 <?xml version="1.0" ?>
-<robot name="korus_v3" xmlns:xacro="http://www.ros.org/wiki/xacro">
-  <xacro:include filename="$(find korus_meta)/resources/urdf/components/omni_drive_base.urdf.xacro"/>
+<robot name="korus" xmlns:xacro="http://www.ros.org/wiki/xacro">
+  <xacro:include filename="$(find korus_meta)/resources/urdf/components/diff_drive_base.urdf.xacro"/>
   <xacro:include filename="$(find korus_meta)/resources/urdf/components/upper_body.urdf.xacro"/>
   <xacro:include filename="$(find korus_meta)/resources/urdf/components/arm.urdf.xacro"/>
-  <xacro:include filename="$(find korus_meta)/resources/urdf/environment/table.urdf.xacro"/>
   <!-- ************************ Base model ************************* -->
-  <xacro:omni_drive_base parent="local_manip_start" body_mount_link="base_link"/>
+  <xacro:diff_drive_base parent="base_footprint" body_mount_link="base_link"/>
   <!-- ************************ Body model ************************* -->
   <xacro:upper_body body_mount_link="base_link" arm_mount_link="torso_lift_link"/>
   <!-- ************************ Arm model ************************* -->
   <xacro:arm arm_mount_link="torso_lift_link"/>
-  <!-- ************************ Table model ************************* -->
-  <xacro:table parent="local_manip_start"/>
 </robot>

File: korus_meta/resources/urdf/korus_omni_drive.urdf.xacro (robot description, xacro)
@@ -1,4 +1,4 @@
 <?xml version="1.0" ?>
-<robot name="korus_v3" xmlns:xacro="http://www.ros.org/wiki/xacro">
+<robot name="korus" xmlns:xacro="http://www.ros.org/wiki/xacro">
   <xacro:include filename="$(find korus_meta)/resources/urdf/components/omni_drive_base.urdf.xacro"/>
   <xacro:include filename="$(find korus_meta)/resources/urdf/components/upper_body.urdf.xacro"/>

Commit message: korus_meta: adds collada mesh for base

File: korus_meta/resources/urdf/components/diff_drive_base.urdf.xacro (robot description, xacro)
@@ -57,5 +57,5 @@
 		  <visual>
 		    <geometry>
-		      <mesh filename="package://korus_meta/resources/meshes/base_test_model.dae" />
+		      <mesh filename="package://korus_meta/resources/meshes/base.dae" />
 		    </geometry>
 		    <origin xyz="0.0 0.0 0.1045" rpy="0 0 0"/>
