Commit message: korus_meta: adds turret collada mesh

File: korus_meta/resources/urdf/components/hokuyo_lx30_laser.urdf.xacro (robot description, xacro)
@@ -15,19 +15,20 @@
         <inertia ixx="0.0001" ixy="0" ixz="0" iyy="0.000001" iyz="0" izz="0.0001" />
       </inertial>
-      <visual>
-        <geometry>
-           <box size="0.050 0.050 0.0703" />
-   	    </geometry>
-        <origin xyz="0.0 0.0 -0.023" rpy="0 0 0"/>
-        <material name="black">
-          <color rgba="0.1 0.1 0.1 1"/>
-        </material>
-      </visual>
-      <collision>
-        <geometry>
-           <box size="0.050 0.050 0.0703" />
-        </geometry>
-        <origin xyz="0.0 0.0 -0.023" rpy="0 0 0"/>
-      </collision>
+<!-- visual and collision is commented out, since the laser is inside the base -->
+<!--       <visual> -->
+<!--         <geometry> -->
+<!--            <box size="0.050 0.050 0.0703" /> -->
+<!--    	    </geometry> -->
+<!--         <origin xyz="0.0 0.0 -0.023" rpy="0 0 0"/>  -->
+<!--         <material name="black"> -->
+<!--           <color rgba="0.1 0.1 0.1 1"/> -->
+<!--         </material> -->
+<!--       </visual> -->
+<!--       <collision> -->
+<!--         <geometry> -->
+<!--            <box size="0.050 0.050 0.0703" /> -->
+<!--         </geometry> -->
+<!--         <origin xyz="0.0 0.0 -0.023" rpy="0 0 0"/>  -->
+<!--       </collision> -->
     </link>
   </xacro:macro>

File: korus_meta/resources/urdf/components/upper_body.urdf.xacro (robot description, xacro)
@@ -15,7 +15,9 @@
 	    <visual>
 	       <geometry>
-	        <cylinder length="0.025" radius="0.278"/>
+<!-- 	        <cylinder length="0.025" radius="0.278"/> -->
+          <mesh filename="package://korus_meta/resources/meshes/turret_test_model_02.dae" />
 	      </geometry>
-	      <origin xyz="0.0 0.0 0.0" rpy="0 0 0"/>
+        <origin xyz="0.0 0.0 0.45885" rpy="0 0 0"/>
+<!-- 	      <origin xyz="0.0 0.0 0.0" rpy="0 0 0"/> -->
 	      <xacro:insert_block name="material_white" />
 	    </visual>
@@ -34,16 +36,17 @@
 	  </joint>
 	  <link name="turret_link">
-	    <visual>
-	      <geometry>
+<!-- 	    <visual> -->
+<!-- 	      <geometry> -->
+<!--            <box size="0.204 0.25746 0.57888" /> -->
+<!-- 	      </geometry> -->
+<!--         <origin xyz="0.0 0.0 0.30194" rpy="0.0 0.0 0.0"/> -->
+<!-- 	      <xacro:insert_block name="material_white" /> -->
+<!-- 	    </visual> -->
+      <collision>
+        <geometry>
            <box size="0.204 0.25746 0.57888" />
-	      </geometry>
+        </geometry>
         <origin xyz="0.0 0.0 0.30194" rpy="0.0 0.0 0.0"/>
-	      <xacro:insert_block name="material_white" />
-	    </visual>
-      <collision>
-        <geometry>
-           <box size="0.204 0.25746 0.57888" />
-        </geometry>
-        <origin xyz="0.0 0.0 0.30194" rpy="0.0 0.0 0.0"/>
+        <xacro:insert_block name="material_white" />
        </collision>
 	  </link>
@@ -69,11 +72,11 @@
 	  </joint>
 	  <link name="neck_link">
-	    <visual>
-	      <geometry>
-          <box size="0.030 0.060 0.23262"/>
-	      </geometry>
-	      <origin xyz="0.0 0.0 0.11631" rpy="0 0 0"/>
-	      <xacro:insert_block name="material_white"/>
-	    </visual>
+<!-- 	    <visual> -->
+<!-- 	      <geometry> -->
+<!--           <box size="0.030 0.060 0.23262"/> -->
+<!-- 	      </geometry> -->
+<!-- 	      <origin xyz="0.0 0.0 0.11631" rpy="0 0 0"/> -->
+<!-- 	      <xacro:insert_block name="material_white"/> -->
+<!-- 	    </visual> -->
       <collision>
         <geometry>
@@ -89,11 +92,11 @@
     </joint>
     <link name="tablet_link">
-      <visual>
-        <geometry>
-          <box size="0.022 0.270 0.1812"/>
-        </geometry>
-        <origin xyz="0.0 0.0 0.0" rpy="0.0 0.0 0.0"/>
-        <xacro:insert_block name="material_black" />
-      </visual>
+<!--       <visual> -->
+<!--         <geometry> -->
+<!--           <box size="0.022 0.270 0.1812"/> -->
+<!--         </geometry> -->
+<!--         <origin xyz="0.0 0.0 0.0" rpy="0.0 0.0 0.0"/> -->
+<!--         <xacro:insert_block name="material_black" /> -->
+<!--       </visual> -->
       <collision>
         <geometry>
@@ -110,11 +113,11 @@
     </joint>
     <link name="head_link">
-      <visual>
-        <geometry>
-          <box size="0.227 0.11872 0.0645" />
-        </geometry>
-        <origin xyz="0.0495 0.0 0.03225" rpy="0.0 0.0 0.0"/>
-        <xacro:insert_block name="material_white" />
-      </visual>
+<!--       <visual> -->
+<!--         <geometry> -->
+<!--           <box size="0.227 0.11872 0.0645" /> -->
+<!--         </geometry> -->
+<!--         <origin xyz="0.0495 0.0 0.03225" rpy="0.0 0.0 0.0"/> -->
+<!--         <xacro:insert_block name="material_white" /> -->
+<!--       </visual> -->
       <collision>
         <geometry>
@@ -130,11 +133,11 @@
     </joint>
     <link name="stargazer_link">
-      <visual>
-        <geometry>
-          <box size="0.09065 0.090 0.0417" />
-        </geometry>
-        <origin xyz="0.02133 0.0 -0.0175" rpy="0.0 0.0 0.0"/>
-        <xacro:insert_block name="material_white" />
-      </visual>
+<!--       <visual> -->
+<!--         <geometry> -->
+<!--           <box size="0.09065 0.090 0.0417" /> -->
+<!--         </geometry> -->
+<!--         <origin xyz="0.02133 0.0 -0.0175" rpy="0.0 0.0 0.0"/> -->
+<!--         <xacro:insert_block name="material_white" /> -->
+<!--       </visual> -->
       <collision>
         <geometry>
