Commit message: updates and cleans urdf descriptions

File: korus_meta/resources/urdf/components/arm.urdf.xacro (robot description, xacro)
@@ -1,7 +1,7 @@
 <?xml version="1.0" ?>
-<robot xmlns:xacro="http://www.ros.org/wiki/xacro" name="korus_3DOF_arm">
-  <include filename="$(find korus_meta)/resources/urdf/materials.urdf.xacro"/>
+<robot xmlns:xacro="http://www.ros.org/wiki/xacro">
+  <xacro:include filename="$(find korus_meta)/resources/urdf/materials.urdf.xacro"/>
   <!-- ************************ Arm macro ************************* -->
-  <xacro:macro name="korus_3DOF_arm" params="arm_mount_link">
+  <xacro:macro name="arm" params="arm_mount_link">
     <joint name="arm_mount" type="fixed">
       <parent link="${arm_mount_link}"/>

File: korus_meta/resources/urdf/components/diff_drive_base.urdf.xacro (robot description, xacro)
@@ -1,4 +1,4 @@
 <?xml version="1.0" ?>
-<robot xmlns:xacro="http://www.ros.org/wiki/xacro" name="diff_drive_base">
+<robot xmlns:xacro="http://www.ros.org/wiki/xacro">
   <xacro:include filename="$(find korus_meta)/resources/urdf/materials.urdf.xacro"/>
   <xacro:include filename="$(find korus_meta)/resources/urdf/hokuyo_lx30_laser.urdf.xacro"/>

File: korus_meta/resources/urdf/components/hokuyo_lx30_laser.gazebo.xacro (robot description, xacro)
@@ -1,8 +1,5 @@
 <?xml version="1.0"?>
 <!--  Move this to a ycs_device_descriptions package -->
-<robot xmlns:sensor="http://playerstage.sourceforge.net/gazebo/xmlschema/#sensor"
-       xmlns:controller="http://playerstage.sourceforge.net/gazebo/xmlschema/#controller"
-       xmlns:interface="http://playerstage.sourceforge.net/gazebo/xmlschema/#interface"
-       xmlns:xacro="http://ros.org/wiki/xacro">
+<robot xmlns:xacro="http://ros.org/wiki/xacro">
   <xacro:property name="hokuyo_lx30_laser_gazebo_pi" value="3.1415926535897931" />
   <xacro:macro name="hokuyo_lx30_laser_gazebo" params="name ros_topic update_rate min_angle max_angle">

File: korus_meta/resources/urdf/components/hokuyo_lx30_laser.urdf.xacro (robot description, xacro)
@@ -1,9 +1,6 @@
 <?xml version="1.0"?>
 <!--  Move this to a ycs_device_descriptions package -->
-<robot xmlns:sensor="http://playerstage.sourceforge.net/gazebo/xmlschema/#sensor"
-       xmlns:controller="http://playerstage.sourceforge.net/gazebo/xmlschema/#controller"
-       xmlns:interface="http://playerstage.sourceforge.net/gazebo/xmlschema/#interface"
-       xmlns:xacro="http://ros.org/wiki/xacro">
-  <include filename="$(find korus_meta)/resources/urdf/hokuyo_lx30_laser.gazebo.xacro" />
+<robot xmlns:xacro="http://ros.org/wiki/xacro">
+  <xacro:include filename="$(find korus_meta)/resources/urdf/hokuyo_lx30_laser.gazebo.xacro" />
   <xacro:macro name="hokuyo_lx30_laser" params="name parent *origin ros_topic update_rate min_angle max_angle">
     <joint name="${name}_joint" type="fixed">

File: korus_meta/resources/urdf/components/materials.urdf.xacro (robot description, xacro)
@@ -1,4 +1,4 @@
 <?xml version="1.0" ?>
-<robot xmlns:xacro="http://www.ros.org/wiki/xacro" name="materials">
+<robot xmlns:xacro="http://www.ros.org/wiki/xacro">
 	<!-- ************************ Properties ************************** -->
 	<xacro:property name="pi" value="3.1415926535897931" />

File: korus_meta/resources/urdf/components/omni_drive_base.urdf.xacro (robot description, xacro)
@@ -1,6 +1,5 @@
 <?xml version="1.0" ?>
-<robot xmlns:xacro="http://www.ros.org/wiki/xacro" name="omni_drive_base">
+<robot xmlns:xacro="http://www.ros.org/wiki/xacro">
   <xacro:include filename="$(find korus_meta)/resources/urdf/materials.urdf.xacro"/>
-  <!-- ************************** TODO!!! ************************** -->
   <!-- ************************** Properties ************************** -->
   <xacro:property name="wheel_bias" value="0.450"/>
@@ -30,8 +29,26 @@
   <xacro:macro name="omni_drive_base" params="parent body_mount_link">
     <link name="${parent}"/>
-    <joint name="base_joint" type="fixed">
+    <joint name="base_position_x" type="prismatic">
       <parent link="${parent}"/>
+      <child link="base_position_x_link"/>
+      <origin rpy="0 0 0" xyz="0.0 0.0 0.0"/>
+      <axis xyz="1 0 0"/>
+      <limit effort="10" lower="-2.0" upper="2.0" velocity="1.0"/>
+    </joint>
+    <link name="base_position_x_link"/>
+    <joint name="base_position_y" type="prismatic">
+      <parent link="base_position_x_link"/>
+      <child link="base_position_y_link"/>
+      <origin rpy="0 0 0" xyz="0.0 0.0 0.0"/>
+      <axis xyz="0 1 0"/>
+      <limit effort="10" lower="-2.0" upper="2.0" velocity="1.0"/>
+    </joint>
+    <link name="base_position_y_link"/>
+    <joint name="base_heading" type="revolute">
+      <parent link="base_position_y_link"/>
       <child link="${body_mount_link}"/>
       <origin rpy="0 0 0" xyz="0.0 0.0 0.075"/>
+      <axis xyz="0 0 1"/>
+      <limit effort="10" lower="-${pi}" upper="${pi}" velocity="1.0"/>
     </joint>
     <link name="${body_mount_link}">
@@ -51,6 +68,6 @@
       </collision>
     </link>
-    <xacro:wheel name="wheel_left" parent="${body_mount_link}" length="0.03" radius="${wheel_radius}" off_x="0.0" off_y="${wheel_bias/2}" off_z="0.0" type="continuous"/>
-    <xacro:wheel name="wheel_right" parent="${body_mount_link}" length="0.03" radius="${wheel_radius}" off_x="0.0" off_y="-${wheel_bias/2}" off_z="0.0" type="continuous"/>
+    <xacro:wheel name="wheel_left" parent="${body_mount_link}" length="0.03" radius="${wheel_radius}" off_x="0.0" off_y="${wheel_bias/2}" off_z="0.0" type="fixed"/>
+    <xacro:wheel name="wheel_right" parent="${body_mount_link}" length="0.03" radius="${wheel_radius}" off_x="0.0" off_y="-${wheel_bias/2}" off_z="0.0" type="fixed"/>
     <xacro:wheel name="caster_front_left" parent="${body_mount_link}" length="0.02" radius="${caster_wheel_radius}" off_x="0.18" off_y="${caster_wheel_bias/2}" off_z="-0.035" type="fixed"/>
     <xacro:wheel name="caster_front_right" parent="${body_mount_link}" length="0.02" radius="${caster_wheel_radius}" off_x="0.18" off_y="-${caster_wheel_bias/2}" off_z="-0.035" type="fixed"/>

File: korus_meta/resources/urdf/components/upper_body.urdf.xacro (robot description, xacro)
@@ -1,7 +1,7 @@
 <?xml version="1.0" ?>
-<robot xmlns:xacro="http://www.ros.org/wiki/xacro" name="korus_v3_body">
-  <include filename="$(find korus_meta)/resources/urdf/materials.urdf.xacro"/>
+<robot xmlns:xacro="http://www.ros.org/wiki/xacro">
+  <xacro:include filename="$(find korus_meta)/resources/urdf/materials.urdf.xacro"/>
   <!-- ************************** Robot body macro ************************** -->
-  <xacro:macro name="korus_v3_body" params="body_mount_link arm_mount_link">
+  <xacro:macro name="upper_body" params="body_mount_link arm_mount_link">
     <!-- ************************** Torso *************************** -->
 	  <joint name="torso_turn" type="revolute">

File: korus_meta/resources/urdf/korus_v3_all.urdf.xacro (robot description, xacro)
@@ -1,41 +1,15 @@
 <?xml version="1.0" ?>
-<robot xmlns:xacro="http://www.ros.org/wiki/xacro" name="korus_v3">
-  <xacro:include filename="$(find korus_meta)/resources/urdf/kinematics_base.urdf.xacro"/>
-  <xacro:include filename="$(find korus_meta)/resources/urdf/diff_drive_base.urdf.xacro"/>
-  <xacro:include filename="$(find korus_meta)/resources/urdf/omni_drive_base.urdf.xacro"/>
-  <xacro:include filename="$(find korus_meta)/resources/urdf/korus_v3_body.urdf.xacro"/>
-  <xacro:include filename="$(find korus_meta)/resources/urdf/korus_3DOF_arm.urdf.xacro"/>
-  <xacro:include filename="$(find korus_meta)/resources/urdf/table.urdf.xacro"/>
+<robot name="korus_v3" xmlns:xacro="http://www.ros.org/wiki/xacro">
+  <xacro:include filename="$(find korus_meta)/resources/urdf/components/omni_drive_base.urdf.xacro"/>
+  <xacro:include filename="$(find korus_meta)/resources/urdf/components/upper_body.urdf.xacro"/>
+  <xacro:include filename="$(find korus_meta)/resources/urdf/components/arm.urdf.xacro"/>
+  <xacro:include filename="$(find korus_meta)/resources/urdf/components/table.urdf.xacro"/>
   <!-- ************************ Base model ************************* -->
-  <xacro:kinematics_base parent="local_manip_start" body_mount_link="base_link"/>
-<!--   <xacro:diff_drive_base parent="base_footprint" body_mount_link="base_link"/> -->
-<!--   <xacro:omni_drive_base parent="base_footprint" body_mount_link="base_link"/> -->
+  <xacro:omni_drive_base parent="local_manip_start" body_mount_link="base_link"/>
   <!-- ************************ Body model ************************* -->
-  <xacro:korus_v3_body body_mount_link="base_link" arm_mount_link="torso_lift_link"/>
+  <xacro:upper_body body_mount_link="base_link" arm_mount_link="torso_lift_link"/>
   <!-- ************************ Arm model ************************* -->
-  <xacro:korus_3DOF_arm arm_mount_link="torso_lift_link"/>
+  <xacro:arm arm_mount_link="torso_lift_link"/>
   <!-- ************************ Table model ************************* -->
   <xacro:table parent="local_manip_start"/>
-  <!-- ************************ Object on floor ************************* -->
-<!--   <joint name="floor_object" type="fixed"> -->
-<!--     <parent link="local_manip_start"/> -->
-<!--     <child link="floor_object_link"/> -->
-<!--     <origin xyz="-0.3 0.0 0.0" rpy="0 0 0" /> -->
-<!--   </joint> -->
-<!-- 	<link name="floor_object_link"> -->
-<!-- 	  <visual> -->
-<!-- 	    <geometry> -->
-<!-- 	      <box size="0.08 0.08 0.15"/> -->
-<!-- 	    </geometry> -->
-<!-- 	    <origin xyz="0.0 0.0 0.075" rpy="0 0 0"/> -->
-<!-- 	    <xacro:insert_block name="material_green" /> -->
-<!-- 	  </visual> -->
-<!-- 	  <collision> -->
-<!-- 	    <geometry> -->
-<!-- 	      <box size="0.08 0.08 0.15"/> -->
-<!-- 	    </geometry> -->
-<!-- 	    <origin xyz="0.0 0.0 0.075" rpy="0 0 0"/> -->
-<!-- 	    <xacro:insert_block name="material_green" />   -->
-<!-- 	  </collision> -->
-<!-- 	</link>   -->
 </robot>

File: korus_meta/resources/urdf/korus_v3_diff_drive.urdf.xacro (robot description, xacro)
@@ -1,12 +1,12 @@
 <?xml version="1.0" ?>
-<robot xmlns:xacro="http://www.ros.org/wiki/xacro" name="korus_v3">
-  <xacro:include filename="$(find korus_meta)/resources/urdf/diff_drive_base.urdf.xacro"/>
-  <xacro:include filename="$(find korus_meta)/resources/urdf/korus_v3_body.urdf.xacro"/>
-  <xacro:include filename="$(find korus_meta)/resources/urdf/korus_3DOF_arm.urdf.xacro"/>
+<robot name="korus_v3" xmlns:xacro="http://www.ros.org/wiki/xacro">
+  <xacro:include filename="$(find korus_meta)/resources/urdf/components/diff_drive_base.urdf.xacro"/>
+  <xacro:include filename="$(find korus_meta)/resources/urdf/components/upper_body.urdf.xacro"/>
+  <xacro:include filename="$(find korus_meta)/resources/urdf/components/arm.urdf.xacro"/>
   <!-- ************************ Base model ************************* -->
   <xacro:diff_drive_base parent="base_footprint" body_mount_link="base_link"/>
   <!-- ************************ Body model ************************* -->
-  <xacro:korus_v3_body body_mount_link="base_link" arm_mount_link="torso_lift_link"/>
+  <xacro:upper_body body_mount_link="base_link" arm_mount_link="torso_lift_link"/>
   <!-- ************************ Arm model ************************* -->
-	<xacro:korus_3DOF_arm arm_mount_link="torso_lift_link"/>
+  <xacro:arm arm_mount_link="torso_lift_link"/>
 </robot>

File: korus_meta/resources/urdf/korus_v3_omni_drive.urdf.xacro (robot description, xacro)
@@ -1,12 +1,12 @@
 <?xml version="1.0" ?>
-<robot xmlns:xacro="http://www.ros.org/wiki/xacro" name="korus_v3">
-  <xacro:include filename="$(find korus_meta)/resources/urdf/omni_drive_base.urdf.xacro"/>
-  <xacro:include filename="$(find korus_meta)/resources/urdf/korus_v3_body.urdf.xacro"/>
-  <xacro:include filename="$(find korus_meta)/resources/urdf/korus_3DOF_arm.urdf.xacro"/>
+<robot name="korus_v3" xmlns:xacro="http://www.ros.org/wiki/xacro">
+  <xacro:include filename="$(find korus_meta)/resources/urdf/components/omni_drive_base.urdf.xacro"/>
+  <xacro:include filename="$(find korus_meta)/resources/urdf/components/upper_body.urdf.xacro"/>
+  <xacro:include filename="$(find korus_meta)/resources/urdf/components/arm.urdf.xacro"/>
   <!-- ************************ Base model ************************* -->
-  <xacro:omni_drive_base parent="base_footprint" body_mount_link="base_link"/>
+  <xacro:omni_drive_base parent="local_manip_start" body_mount_link="base_link"/>
   <!-- ************************ Body model ************************* -->
-  <xacro:korus_v3_body body_mount_link="base_link" arm_mount_link="torso_lift_link"/>
+  <xacro:upper_body body_mount_link="base_link" arm_mount_link="torso_lift_link"/>
   <!-- ************************ Arm model ************************* -->
-	<xacro:korus_3DOF_arm arm_mount_link="torso_lift_link"/>
+	<xacro:arm arm_mount_link="torso_lift_link"/>
 </robot>

Commit message: new meshes for URDF

File: korus_meta/resources/urdf/components/arm.urdf.xacro (robot description, xacro)
@@ -12,7 +12,8 @@
       <visual>
         <geometry>
-          <box size="0.122 0.254 0.131"/>
-        </geometry>
-        <origin xyz="-0.020 0.070 -0.0655" rpy="0 0 0"/>
+<!--           <box size="0.122 0.254 0.131"/> -->
+          <mesh filename="package://korus_meta/resources/meshes/shoulder.dae" />
+        </geometry>
+        <origin xyz="-0.020 0.070 -0.034" rpy="${-pi/2} 0 0"/>
         <xacro:insert_block name="material_white"/>
       </visual>

File: korus_meta/resources/urdf/components/upper_body.urdf.xacro (robot description, xacro)
@@ -16,5 +16,5 @@
 	       <geometry>
 <!-- 	        <cylinder length="0.025" radius="0.278"/> -->
-          <mesh filename="package://korus_meta/resources/meshes/turret_test_model_02.dae" />
+          <mesh filename="package://korus_meta/resources/meshes/turret.dae" />
 	      </geometry>
         <origin xyz="0.0 0.0 0.45885" rpy="0 0 0"/>
@@ -157,5 +157,6 @@
       <visual>
         <geometry>
-          <box size="0.1122 0.090 0.0417"/>
+<!--           <box size="0.1122 0.090 0.0417"/> -->
+          <mesh filename="package://korus_meta/resources/meshes/head_pan.dae" />
         </geometry>
         <origin xyz="-0.0339 0.0 0.02085" rpy="0.0 0.0 0.0"/>
@@ -172,15 +173,9 @@
       <parent link="head_pan_link"/>
       <child link="head_tilt_link"/>
-      <origin xyz="0.028 0.0 0.0275" rpy="${pi/2} 0 0"/> <!-- x original 0.013 -->
+      <origin xyz="0.01 0.0 0.025" rpy="${pi/2} 0 0"/> <!-- x original 0.013 -->
       <axis xyz="0 0 1"/>
       <limit effort="9.0" lower="${-92*rad}" upper="${32*rad}" velocity="${476*rad}"/>
     </joint>
     <link name="head_tilt_link"/>
-    <joint name="head_tilt_fixed" type="fixed">
-      <parent link="head_link"/>
-      <child link="head_tilt_fixed_link"/>
-      <origin xyz="0.146 0.0 0.092" rpy="${pi/2} 0 0"/>
-    </joint>
-    <link name="head_tilt_fixed_link"/>
     <!-- Frames published by openni_launch expect <camera name>_link tf
          as parent, so we publish this fake link just to satisfy it -->
@@ -188,14 +183,17 @@
       <parent link="head_tilt_link"/>
       <child link="sensor_3d_link"/>
-      <!-- adds 2 deg to yaw, because the xtion is mounted on its surface which is inclined (approx. 2 deg) -->
-      <origin xyz="0.0 0.0 0.0" rpy="${-pi/2} 0 0.035"/>
+      <!-- IHeartRobotics: adds 2 deg to yaw, because the xtion is mounted on its surface which is inclined (approx. 2 deg) -->
+<!--       <origin xyz="0.0 0.0 0.0" rpy="${-pi/2} 0 0.035"/> -->
+      <origin xyz="0.0 0.0 0.0" rpy="${-pi/2} 0 0.0"/>
     </joint>
     <link name="sensor_3d_link">
       <visual>
-        <origin xyz="0.0075 0.0 0.0315" rpy="${pi/2} 0 ${pi/2}" />
         <geometry>
            <!-- Thank you IHeartRobotics for the Xtion mesh! -->
-           <mesh filename="package://korus_meta/resources/meshes/asus_xtion_pro_live.dae" scale="0.001 0.001 0.001"/>
-        </geometry>
+<!--            <mesh filename="package://korus_meta/resources/meshes/asus_xtion_pro_live.dae" scale="0.001 0.001 0.001"/> -->
+           <mesh filename="package://korus_meta/resources/meshes/xtionpro_w_mount.dae"/>
+        </geometry>
+<!--         <origin xyz="0.0075 0.0 0.0315" rpy="${pi/2} 0 ${pi/2}" /> -->
+        <origin xyz="0.0 0.0 0.0225" rpy="0 0 0" />
         <xacro:insert_block name="material_black"/>
       </visual>
