Commit message: korus_meta: adds arm meshes and fixes collision models (colour issue)

File: korus_meta/resources/urdf/components/arm.urdf.xacro (robot description, xacro)
@@ -12,5 +12,4 @@
       <visual>
         <geometry>
-<!--           <box size="0.122 0.254 0.131"/> -->
           <mesh filename="package://korus_meta/resources/meshes/shoulder.dae" />
         </geometry>
@@ -35,7 +34,7 @@
 	    <visual>
 	      <geometry>
-	        <box size="0.378 0.095 0.055"/>
+          <mesh filename="package://korus_meta/resources/meshes/upper_arm.dae" />
 	      </geometry>
-	      <origin xyz="0.1415 0.0 0.0275" rpy="0 0 0"/>
+	      <origin xyz="0.1425 0.001 0.0275" rpy="${pi/2} ${pi} ${pi/2}"/>
 	      <xacro:insert_block name="material_white" />
 	    </visual>
@@ -44,5 +43,5 @@
           <box size="0.378 0.095 0.055"/>
         </geometry>
-        <origin xyz="0.1415 0.0 0.0275" rpy="0 0 0"/>
+        <origin xyz="0.145 0.0 0.028" rpy="0 0 0"/>
        </collision>
 	  </link>
@@ -57,7 +56,7 @@
 	    <visual>
 	      <geometry>
-	        <box size="0.477 0.095 0.057"/>
+          <mesh filename="package://korus_meta/resources/meshes/lower_arm.dae" />
 	      </geometry>
-	      <origin xyz="0.19426 0.00 0.0285" rpy="0 0 0"/>
+	      <origin xyz="0.19 0.002 0.027" rpy="${pi/2} ${pi} ${pi/2}"/>
 	      <xacro:insert_block name="material_white" />
 	    </visual>
@@ -76,33 +75,25 @@
 	    <limit effort="51.0" lower="${-100*rad}" upper="${100*rad}" velocity="${72.5*rad}"/>
 	  </joint>
-	  <link name="wrist_link">
-	    <visual>
-	      <geometry>
-          <cylinder length="0.0854" radius="0.038"/>
-	      </geometry>
-	      <origin xyz="0.0 0.0 -0.0427" rpy="0 0 0"/>
-	      <xacro:insert_block name="material_white"/>
-	    </visual>
-      <collision>
-        <geometry>
-          <cylinder length="0.0854" radius="0.038"/>
-        </geometry>
-        <origin xyz="0.0 0.0 -0.0427" rpy="0 0 0"/>
-      </collision>
-	  </link>
+	  <link name="wrist_link"/>
   	<!--   Endeffector (gripper)  -->
 	  <joint name="palm" type="fixed">
 	    <parent link="wrist_link"/>
 	    <child link="palm_link"/>
-	    <origin xyz="0.0 0.0 -0.045" rpy="0 0 0"/>
+	    <origin xyz="0.0 0.0 -0.0425" rpy="0 0 0"/>
 	  </joint>
 	  <link name="palm_link">
 	    <visual>
 	      <geometry>
-	        <box size="0.1044 0.077 0.0804"/>
+          <mesh filename="package://korus_meta/resources/meshes/palm.dae" />
 	      </geometry>
-	      <origin xyz="0.0522 0.0 0.0" rpy="0 0 0"/>
-        <xacro:insert_block name="material_white"/>
-      </visual>
+	      <origin xyz="0.0395 0.001 0.0" rpy="${-pi/2} 0 0"/>
+        <xacro:insert_block name="material_white"/>
+      </visual>
+      <collision>
+        <geometry>
+          <cylinder length="0.0854" radius="0.038"/>
+        </geometry>
+        <origin xyz="0.0 0.0 0.0035" rpy="0 0 0"/>
+      </collision>
       <collision>
         <geometry>
@@ -135,7 +126,7 @@
 	  <link name="finger_left_knuckle_1_link">
       <visual>
-	      <geometry>
-	        <box size="0.0595 0.0247 0.0306"/>
-	      </geometry>
+        <geometry>
+          <mesh filename="package://korus_meta/resources/meshes/finger01.dae" />
+        </geometry>
 	      <origin xyz="0.02975 0.0 0.0" rpy="0 0 0"/>
 	      <xacro:insert_block name="material_white"/>
@@ -158,5 +149,5 @@
       <visual>
         <geometry>
-          <box size="0.065 0.0247 0.0306"/>
+          <mesh filename="package://korus_meta/resources/meshes/finger02.dae" />
         </geometry>
         <origin xyz="0.0325 0.0 0.0" rpy="0 0 0"/>
@@ -186,5 +177,5 @@
       <visual>
         <geometry>
-          <box size="0.0595 0.0247 0.0306"/>
+          <mesh filename="package://korus_meta/resources/meshes/finger01.dae" />
         </geometry>
         <origin xyz="0.02975 0.0 0.0" rpy="0 0 0"/>
@@ -208,5 +199,5 @@
       <visual>
         <geometry>
-          <box size="0.065 0.0247 0.0306"/>
+          <mesh filename="package://korus_meta/resources/meshes/finger02.dae" />
         </geometry>
         <origin xyz="0.0325 0.0 0.0" rpy="0 0 0"/>

File: korus_meta/resources/urdf/components/diff_drive_base.urdf.xacro (robot description, xacro)
@@ -35,13 +35,13 @@
     </joint>
     <link name="${name}_link">
-      <visual>
-        <geometry>
-          <cylinder length="${length}" radius="${radius}"/>
-        </geometry>
-        <origin rpy="0 ${pi/2} 0" xyz="0 0 0"/>
-        <material name="black">
-          <color rgba="0.1 0.1 0.1 1"/>
-        </material>
-      </visual>
+<!--       <visual> -->
+<!--         <geometry> -->
+<!--           <cylinder length="${length}" radius="${radius}"/> -->
+<!--         </geometry> -->
+<!--         <origin rpy="0 ${pi/2} 0" xyz="0 0 0"/> -->
+<!--         <material name="black"> -->
+<!--           <color rgba="0.1 0.1 0.1 1"/> -->
+<!--         </material> -->
+<!--       </visual> -->
     </link>
   </xacro:macro>

File: korus_meta/resources/urdf/components/upper_body.urdf.xacro (robot description, xacro)
@@ -14,18 +14,45 @@
 	  <link name="torso_link">
 	    <visual>
-	       <geometry>
-<!-- 	        <cylinder length="0.025" radius="0.278"/> -->
+	      <geometry>
           <mesh filename="package://korus_meta/resources/meshes/turret.dae" />
 	      </geometry>
         <origin xyz="0.0 0.0 0.45885" rpy="0 0 0"/>
-<!-- 	      <origin xyz="0.0 0.0 0.0" rpy="0 0 0"/> -->
 	      <xacro:insert_block name="material_white" />
 	    </visual>
-      <collision>
+      <collision> <!-- torso turn disk -->
          <geometry>
           <cylinder length="0.025" radius="0.278"/>
         </geometry>
         <origin xyz="0.0 0.0 0.0" rpy="0 0 0"/>
-        <xacro:insert_block name="material_white" />
+      </collision>
+      <collision> <!-- back -->
+        <geometry>
+           <box size="0.204 0.25746 0.57888" />
+        </geometry>
+        <origin xyz="-0.13786 0.0 0.30194" rpy="0 0 0"/>
+      </collision>
+      <collision> <!-- neck -->
+        <geometry>
+          <box size="0.030 0.060 0.23262"/>
+        </geometry>
+        <origin xyz="-0.12536  0.0 0.70769" rpy="0 0 0"/>
+      </collision>
+      <collision> <!-- tablet -->
+        <geometry>
+          <box size="0.022 0.270 0.1812"/>
+        </geometry>
+        <origin xyz="-0.04036 0.0 0.6495" rpy="0 0 0"/>
+      </collision>
+      <collision> <!-- head -->
+        <geometry>
+          <box size="0.227 0.11872 0.0645" />
+        </geometry>
+        <origin xyz="-0.07586 0.0 0.85625" rpy="0 0 0"/>
+      </collision>
+      <collision> <!-- stargazer -->
+        <geometry>
+          <box size="0.09065 0.090 0.0417" />
+        </geometry>
+        <origin xyz="-0.14403 0.0 0.909" rpy="0 0 0"/>
       </collision>
 	  </link>
@@ -35,20 +62,5 @@
 	    <origin xyz="-0.13786 0.0 0.0" rpy="0 0 0"/>
 	  </joint>
-	  <link name="turret_link">
-<!-- 	    <visual> -->
-<!-- 	      <geometry> -->
-<!--            <box size="0.204 0.25746 0.57888" /> -->
-<!-- 	      </geometry> -->
-<!--         <origin xyz="0.0 0.0 0.30194" rpy="0.0 0.0 0.0"/> -->
-<!-- 	      <xacro:insert_block name="material_white" /> -->
-<!-- 	    </visual> -->
-      <collision>
-        <geometry>
-           <box size="0.204 0.25746 0.57888" />
-        </geometry>
-        <origin xyz="0.0 0.0 0.30194" rpy="0.0 0.0 0.0"/>
-        <xacro:insert_block name="material_white" />
-       </collision>
-	  </link>
+	  <link name="turret_link"/>
 	  <joint name="torso_lift_offset" type="fixed">
 	    <parent link="turret_link"/>
@@ -69,41 +81,13 @@
 	    <parent link="turret_link"/>
 	    <child link="neck_link"/>
-	    <origin rpy="0 0 0" xyz="0.0125 0.0 0.59138"/>
-	  </joint>
-	  <link name="neck_link">
-<!-- 	    <visual> -->
-<!-- 	      <geometry> -->
-<!--           <box size="0.030 0.060 0.23262"/> -->
-<!-- 	      </geometry> -->
-<!-- 	      <origin xyz="0.0 0.0 0.11631" rpy="0 0 0"/> -->
-<!-- 	      <xacro:insert_block name="material_white"/> -->
-<!-- 	    </visual> -->
-      <collision>
-        <geometry>
-          <box size="0.030 0.060 0.23262"/>
-        </geometry>
-        <origin xyz="0.0 0.0 0.11631" rpy="0 0 0"/>
-      </collision>
-	  </link>
+	    <origin xyz="0.0125 0.0 0.59138" rpy="0 0 0"/>
+	  </joint>
+	  <link name="neck_link"/>
     <joint name="tablet" type="fixed">
       <parent link="neck_link"/>
       <child link="tablet_link"/>
-      <origin rpy="0 0 0" xyz="0.085 0.0 0.05812"/>
-    </joint>
-    <link name="tablet_link">
-<!--       <visual> -->
-<!--         <geometry> -->
-<!--           <box size="0.022 0.270 0.1812"/> -->
-<!--         </geometry> -->
-<!--         <origin xyz="0.0 0.0 0.0" rpy="0.0 0.0 0.0"/> -->
-<!--         <xacro:insert_block name="material_black" /> -->
-<!--       </visual> -->
-      <collision>
-        <geometry>
-          <box size="0.022 0.270 0.1812"/>
-        </geometry>
-        <origin xyz="0.0 0.0 0.0" rpy="0.0 0.0 0.0"/>
-      </collision>
-    </link>
+      <origin xyz="0.085 0.0 0.05812" rpy="0 0 0"/>
+    </joint>
+    <link name="tablet_link"/>
 	  <!-- ************************** Head with ASUS Xtion Pro Live and Stargazer ************************** -->
     <joint name="head" type="fixed">
@@ -112,19 +96,5 @@
       <origin xyz="0.0 0.0 0.23262" rpy="0 0 0"/>
     </joint>
-    <link name="head_link">
-<!--       <visual> -->
-<!--         <geometry> -->
-<!--           <box size="0.227 0.11872 0.0645" /> -->
-<!--         </geometry> -->
-<!--         <origin xyz="0.0495 0.0 0.03225" rpy="0.0 0.0 0.0"/> -->
-<!--         <xacro:insert_block name="material_white" /> -->
-<!--       </visual> -->
-      <collision>
-        <geometry>
-          <box size="0.227 0.11872 0.0645" />
-        </geometry>
-        <origin xyz="0.0495 0.0 0.03225" rpy="0.0 0.0 0.0"/>
-      </collision>
-    </link>
+    <link name="head_link"/>
     <joint name="stargazer" type="fixed">
       <parent link="head_link"/>
@@ -132,19 +102,5 @@
       <origin xyz="-0.040 0.0 0.1025" rpy="0 0 ${pi}"/>
     </joint>
-    <link name="stargazer_link">
-<!--       <visual> -->
-<!--         <geometry> -->
-<!--           <box size="0.09065 0.090 0.0417" /> -->
-<!--         </geometry> -->
-<!--         <origin xyz="0.02133 0.0 -0.0175" rpy="0.0 0.0 0.0"/> -->
-<!--         <xacro:insert_block name="material_white" /> -->
-<!--       </visual> -->
-      <collision>
-        <geometry>
-          <box size="0.09065 0.090 0.0417" />
-        </geometry>
-        <origin xyz="0.02133 0.0 -0.0175" rpy="0.0 0.0 0.0"/>
-      </collision>
-    </link>
+    <link name="stargazer_link"/>
     <joint name="head_pan" type="revolute">
       <parent link="head_link"/>
@@ -157,5 +113,4 @@
       <visual>
         <geometry>
-<!--           <box size="0.1122 0.090 0.0417"/> -->
           <mesh filename="package://korus_meta/resources/meshes/head_pan.dae" />
         </geometry>
@@ -183,5 +138,5 @@
       <parent link="head_tilt_link"/>
       <child link="sensor_3d_link"/>
-      <!-- IHeartRobotics: adds 2 deg to yaw, because the xtion is mounted on its surface which is inclined (approx. 2 deg) -->
+      <!-- adds 2 deg to yaw, because the xtion is mounted on its surface which is inclined (approx. 2 deg) -->
 <!--       <origin xyz="0.0 0.0 0.0" rpy="${-pi/2} 0 0.035"/> -->
       <origin xyz="0.0 0.0 0.0" rpy="${-pi/2} 0 0.0"/>
@@ -190,9 +145,6 @@
       <visual>
         <geometry>
-           <!-- Thank you IHeartRobotics for the Xtion mesh! -->
-<!--            <mesh filename="package://korus_meta/resources/meshes/asus_xtion_pro_live.dae" scale="0.001 0.001 0.001"/> -->
            <mesh filename="package://korus_meta/resources/meshes/xtionpro_w_mount.dae"/>
         </geometry>
-<!--         <origin xyz="0.0075 0.0 0.0315" rpy="${pi/2} 0 ${pi/2}" /> -->
         <origin xyz="0.0 0.0 0.0225" rpy="0 0 0" />
         <xacro:insert_block name="material_black"/>

Commit message: korus_meta: updates for launchers and urdf

File: korus_meta/resources/urdf/components/arm.urdf.xacro (robot description, xacro)
@@ -80,5 +80,5 @@
 	    <parent link="wrist_link"/>
 	    <child link="palm_link"/>
-	    <origin xyz="0.0 0.0 -0.0425" rpy="0 0 0"/>
+	    <origin xyz="0.0 0.0 -0.045" rpy="0 0 0"/>
 	  </joint>
 	  <link name="palm_link">
@@ -87,5 +87,5 @@
           <mesh filename="package://korus_meta/resources/meshes/palm.dae" />
 	      </geometry>
-	      <origin xyz="0.0395 0.001 0.0" rpy="${-pi/2} 0 0"/>
+	      <origin xyz="0.0395 0.001 0.0025" rpy="${-pi/2} 0 0"/>
         <xacro:insert_block name="material_white"/>
       </visual>

File: korus_meta/resources/urdf/components/upper_body.urdf.xacro (robot description, xacro)
@@ -139,6 +139,6 @@
       <child link="sensor_3d_link"/>
       <!-- adds 2 deg to yaw, because the xtion is mounted on its surface which is inclined (approx. 2 deg) -->
-<!--       <origin xyz="0.0 0.0 0.0" rpy="${-pi/2} 0 0.035"/> -->
-      <origin xyz="0.0 0.0 0.0" rpy="${-pi/2} 0 0.0"/>
+      <origin xyz="0.0 0.0 0.0" rpy="${-pi/2} 0 0.035"/>
+<!--       <origin xyz="0.0 0.0 0.0" rpy="${-pi/2} 0 0.0"/>  -->
     </joint>
     <link name="sensor_3d_link">

Commit message: korus_meta: adjusts elbow joint limit

File: korus_meta/resources/urdf/components/arm.urdf.xacro (robot description, xacro)
@@ -51,5 +51,6 @@
 	    <origin xyz="0.283 0.0 0.055" rpy="0 0 0"/>
 	    <axis xyz="0 0 1"/>
-	    <limit effort="200.0" lower="${-200*rad}" upper="${92*rad}" velocity="${91*rad}"/>
+<!--       <limit effort="200.0" lower="${-200*rad}" upper="${92*rad}" velocity="${91*rad}"/> -->
+	    <limit effort="200.0" lower="${-190*rad}" upper="${92*rad}" velocity="${91*rad}"/>
 	  </joint>
 	  <link name="lower_arm_link">

Commit message: korus_meta: adds modified gripper finger link

File: korus_meta/resources/urdf/components/arm.urdf.xacro (robot description, xacro)
@@ -200,12 +200,13 @@
       <visual>
         <geometry>
-          <mesh filename="package://korus_meta/resources/meshes/finger02.dae" />
-        </geometry>
-        <origin xyz="0.0325 0.0 0.0" rpy="0 0 0"/>
-        <xacro:insert_block name="material_white"/>
-      </visual>
-      <collision>
-        <geometry>
-          <box size="0.065 0.0247 0.0306"/>
+<!--           <mesh filename="package://korus_meta/resources/meshes/finger02.dae" /> -->
+          <box size="0.065 0.0247 0.08"/>
+        </geometry>
+        <origin xyz="0.0325 0.0 0.0" rpy="0 0 0"/>
+        <xacro:insert_block name="material_white"/>
+      </visual>
+      <collision>
+        <geometry>
+          <box size="0.065 0.0247 0.08"/>
         </geometry>
         <origin xyz="0.0325 0.0 0.0" rpy="0 0 0"/>

Commit message: korus_meta: fixes elbow lower joint limit

File: korus_meta/resources/urdf/components/arm.urdf.xacro (robot description, xacro)
@@ -51,6 +51,5 @@
 	    <origin xyz="0.283 0.0 0.055" rpy="0 0 0"/>
 	    <axis xyz="0 0 1"/>
-<!--       <limit effort="200.0" lower="${-200*rad}" upper="${92*rad}" velocity="${91*rad}"/> -->
-	    <limit effort="200.0" lower="${-190*rad}" upper="${92*rad}" velocity="${91*rad}"/>
+	    <limit effort="200.0" lower="${-180*rad}" upper="${92*rad}" velocity="${91*rad}"/>
 	  </joint>
 	  <link name="lower_arm_link">

Commit message: korus_meta: changes wrist camera model description for working around urdf to collada converter bug

File: korus_meta/resources/urdf/components/arm.urdf.xacro (robot description, xacro)
@@ -226,5 +226,5 @@
       <visual>
         <geometry>
-          <cylinder length="0.01" radius="0.005"/>
+          <cylinder length="0.01" radius="0.01"/>
         </geometry>
         <origin xyz="0.0 0.0 0.0" rpy="0 0 0"/>
@@ -233,8 +233,7 @@
       <collision>
         <geometry>
-          <cylinder length="0.01" radius="0.005"/>
+          <cylinder length="0.01" radius="0.01"/>
         </geometry>
         <origin xyz="0.0 0.0 0.0" rpy="0 0 0"/>
-        <xacro:insert_block name="material_black"/>
       </collision>
     </link>
