Commit message: korus_meta: fixes 3d sensor's rgb frame position

File: korus_meta/resources/urdf/components/upper_body.urdf.xacro (robot description, xacro)
@@ -162,11 +162,5 @@
       <child link="sensor_3d_depth_frame" />
     </joint>
-    <link name="sensor_3d_depth_frame">
-      <inertial>
-        <mass value="0.01" />
-        <origin xyz="0 0 0" />
-        <inertia ixx="0.001" ixy="0.0" ixz="0.0"
-                 iyy="0.001" iyz="0.0" izz="0.001" />
-      </inertial>
+    <link name="sensor_3d_depth_frame"/>>
     </link>
     <joint name="sensor_3d_depth_optical_joint" type="fixed">
@@ -175,25 +169,11 @@
       <child link="sensor_3d_depth_optical_frame" />
     </joint>
-    <link name="sensor_3d_depth_optical_frame">
-      <inertial>
-        <mass value="0.001" />
-        <origin xyz="0 0 0" />
-        <inertia ixx="0.0001" ixy="0.0" ixz="0.0"
-                 iyy="0.0001" iyz="0.0" izz="0.0001" />
-      </inertial>
-    </link>
+    <link name="sensor_3d_depth_optical_frame"/>
     <joint name="sensor_3d_rgb_joint" type="fixed">
-      <origin xyz="0.01 0.023 0.0315" rpy="0 -0.017 0" />
+      <origin xyz="0.01 0.005 0.0315" rpy="0 -0.017 0" />
       <parent link="sensor_3d_link" />
       <child link="sensor_3d_rgb_frame" />
     </joint>
-    <link name="sensor_3d_rgb_frame">
-      <inertial>
-        <mass value="0.001" />
-        <origin xyz="0 0 0" />
-        <inertia ixx="0.0001" ixy="0.0" ixz="0.0"
-                 iyy="0.0001" iyz="0.0" izz="0.0001" />
-      </inertial>
-    </link>
+    <link name="sensor_3d_rgb_frame"/>
     <joint name="sensor_3d_rgb_optical_joint" type="fixed">
       <origin xyz="0 0 0" rpy="${-pi/2} 0 ${-pi/2}" />
@@ -201,12 +181,5 @@
       <child link="sensor_3d_rgb_optical_frame" />
     </joint>
-    <link name="sensor_3d_rgb_optical_frame">
-      <inertial>
-        <mass value="0.001" />
-        <origin xyz="0 0 0" />
-        <inertia ixx="0.0001" ixy="0.0" ixz="0.0"
-                 iyy="0.0001" iyz="0.0" izz="0.0001" />
-      </inertial>
-    </link>
+    <link name="sensor_3d_rgb_optical_frame"/>
   </xacro:macro>
 </robot>

Commit message: korus_meta: fixes typo in upper_body.urdf

File: korus_meta/resources/urdf/components/upper_body.urdf.xacro (robot description, xacro)
@@ -162,6 +162,5 @@
       <child link="sensor_3d_depth_frame" />
     </joint>
-    <link name="sensor_3d_depth_frame"/>>
-    </link>
+    <link name="sensor_3d_depth_frame"/>
     <joint name="sensor_3d_depth_optical_joint" type="fixed">
       <origin xyz="0 0 0" rpy="${-pi/2} 0 ${-pi/2}" />

Commit message: Fix mismatched tag

File: korus_meta/resources/urdf/components/upper_body.urdf.xacro (robot description, xacro)
@@ -163,5 +163,4 @@
     </joint>
     <link name="sensor_3d_depth_frame"/>>
-    </link>
     <joint name="sensor_3d_depth_optical_joint" type="fixed">
       <origin xyz="0 0 0" rpy="${-pi/2} 0 ${-pi/2}" />

Commit message: korus_meta: adds launchers for motion retargeting

File: korus_meta/resources/urdf/components/upper_body.urdf.xacro (robot description, xacro)
@@ -138,7 +138,6 @@
       <parent link="head_tilt_link"/>
       <child link="sensor_3d_link"/>
-      <!-- adds 2 deg to yaw, because the xtion is mounted on its surface which is inclined (approx. 2 deg) -->
-      <origin xyz="0.0 0.0 0.0" rpy="${-pi/2} 0 0.035"/>
-<!--       <origin xyz="0.0 0.0 0.0" rpy="${-pi/2} 0 0.0"/>  -->
+      <!-- adds to yaw, because the xtion is mounted on its surface which is inclined (approx. 2 deg) -->
+      <origin xyz="0.0 0.0 0.0" rpy="${-pi/2} 0 0.034"/>
     </joint>
     <link name="sensor_3d_link">
@@ -157,6 +156,12 @@
       </collision>
     </link>
+    <joint name="sensor_3d_fixed" type="fixed"> <!-- used for head pose control -->
+      <parent link="head_link"/>
+      <child link="sensor_3d_fixed_link"/>
+      <origin xyz="0.143 0.0 0.1225" rpy="0 0 0"/>
+    </joint>
+    <link name="sensor_3d_fixed_link"/>
     <joint name="sensor_3d_depth_joint" type="fixed">
-      <origin xyz="0.01 0.0485 0.0315" rpy="0 0.0 0" />
+      <origin xyz="0.019 0.0435 0.0315" rpy="0 0 0" />
       <parent link="sensor_3d_link" />
       <child link="sensor_3d_depth_frame" />
@@ -170,5 +175,6 @@
     <link name="sensor_3d_depth_optical_frame"/>
     <joint name="sensor_3d_rgb_joint" type="fixed">
-      <origin xyz="0.01 0.005 0.0315" rpy="0 -0.017 0" />
+<!--       <origin xyz="0.0175 0.005 0.0315" rpy="0 -0.017 0" /> already applied in the sensor_3d_link -->
+      <origin xyz="0.0 0.015 0.0315" rpy="0 0 0" />
       <parent link="sensor_3d_link" />
       <child link="sensor_3d_rgb_frame" />

Commit message: korus_meta: adds few mods for motion retargeting

File: korus_meta/resources/urdf/components/upper_body.urdf.xacro (robot description, xacro)
@@ -57,4 +57,12 @@
       </collision>
 	  </link>
+    <!-- (Fixed) Reference torso for motion retargeting -->
+    <joint name="torso_mo_ret_joint" type="fixed">
+      <parent link="${body_mount_link}"/>
+      <child link="torso_mo_ret_link"/>
+      <origin rpy="0 0 0" xyz="0.0 0.0 0.2665"/>
+      <axis xyz="0 0 1"/>
+    </joint>
+    <link name="torso_mo_ret_link"/>
 	  <joint name="turret" type="fixed">
 	    <parent link="torso_link"/>
